File: Model 64 Sequencer Cartridge v1.brd (EAGLE design)
At the start: 176.5 x 83.8 mm, 59 parts, among them IC1 68A21, IC2 6850, IC3 27C128, IC4 74LS74N, IC5 4011N, IC6 74LS04N, IC7 74LS04N, IC8 74ALS08N, J1 S-PJ301M, J2 PJ301M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

Commit message: Update to use 6.35mm jacks
Parts:
- J1: value S-PJ301M -> N112BPCX; device thonkiconn_eagle_v5 (2):JACK-3.5-STEREO -> N112BPCX:SWITCHCRAFT_N112BPCX
- J2: value PJ301M -> N111PCX; device thonkiconn:WQP-PJ301M-12_JACK -> N111PCX:SWITCHCRAFT_N111PCX
- moved J2 2.54 mm to (160.0, 71.1), turned to 90 degrees
- moved J1 1.42 mm to (160.0, 15.9), turned to 0 degrees
Connections:
- net GND: now also J1.SLV, J2.SLV; no longer J1.1, J2.3
- net N$33: now also J1.T; no longer J1.3
- net N$35: now also J2.T; no longer J2.1
- net N$38: now also J1.R; no longer J1.2
Routing:
- net GND: track 881.5 -> 863.9 mm
- net N$35: track 25.6 -> 31.8 mm
- net N$40: track 118.3 -> 113.7 mm
- net N$33: track 51.6 -> 49.2 mm
- net N$38: track 37.3 -> 38.0 mm
