File: Model 64 Sequencer Cartridge v1.sch (EAGLE design)
At the start: 55 parts, among them IC1 68A21, IC2 6850, IC3 27C128, IC4 74LS74N, IC5 4011N, IC6 74LS04N, IC7 74LS04N, IC8 74ALS08N, J1 S-PJ301M, J2 PJ301M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

Commit message: Update to use 6.35mm jacks
Parts:
- J1: value S-PJ301M -> N112BPCX; device thonkiconn_eagle_v5 (2):STEREO-PJ301M -> N112BPCX:N112BPCX
- J2: value PJ301M -> N111PCX; device thonkiconn:WQP-PJ301M-12_JACKPJ301M -> N111PCX:N111PCX
Connections:
- net GND: now also J1.SLEEVE, J2.SLEEVE; no longer J1.1, J2.1
- net N$33: now also J1.TIP; no longer J1.3
- net N$35: now also J2.TIP; no longer J2.2
- net N$38: now also J1.RING; no longer J1.2
Changed lines of the file:
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@@
 <part name="P+20" library="supply1" deviceset="+5V" device=""/>
 <part name="C1" library="rcl" deviceset="C-EU" device="050-024X044" value="100n"/>
-<part name="J2" library="thonkiconn" deviceset="WQP-PJ301M-12_JACK" device="PJ301M" value="PJ301M"/>
 <part name="GND7" library="supply1" deviceset="GND" device=""/>
 <part name="R9" library="rcl" deviceset="R-US_" device="0207/12" value="100k"/>
 <part name="R5" library="rcl" deviceset="R-US_" device="0207/12" value="1M"/>
 <part name="P+21" library="supply1" deviceset="+5V" device=""/>
-<part name="J1" library="thonkiconn_eagle_v5 (2)" deviceset="STEREO-PJ301M" device="" value="S-PJ301M"/>
 <part name="GND8" library="supply1" deviceset="GND" device=""/>
 <part name="P+22" library="supply1" deviceset="+5V" device=""/>
@@
 <part name="P+36" library="supply1" deviceset="+5V" device=""/>
 <part name="GND27" library="supply1" deviceset="GND" device=""/>
+<part name="J2" library="N111PCX" deviceset="N111PCX" device=""/>
+<part name="J1" library="N112BPCX" deviceset="N112BPCX" device=""/>
 </parts>
 <sheets>
@@
 <text x="20.32" y="165.1" size="1.778" layer="97">Clock Source</text>
 <text x="7.62" y="127" size="1.778" layer="97">Start/Stop</text>
-<text x="7.62" y="162.56" size="1.778" layer="97">Clock In</text>
+<text x="7.62" y="165.1" size="1.778" layer="97">Clock In</text>
 <text x="294.64" y="124.46" size="1.778" layer="97">Cartridge Connector</text>
 </plain>
@@
 <attribute name="VALUE" x="33.401" y="120.396" size="1.778" layer="96" rot="R270"/>
 </instance>
-<instance part="J2" gate="G$1" x="15.24" y="119.38" smashed="yes" rot="MR0">
-<attribute name="NAME" x="17.78" y="123.444" size="1.778" layer="95" rot="MR0"/>
-<attribute name="VALUE" x="17.78" y="113.284" size="1.778" layer="96" rot="MR0"/>
-</instance>
-<instance part="GND7" gate="1" x="22.86" y="111.76" smashed="yes">
-<attribute name="VALUE" x="20.32" y="109.22" size="1.778" layer="96"/>
+<instance part="GND7" gate="1" x="25.4" y="111.76" smashed="yes">
+<attribute name="VALUE" x="22.86" y="109.22" size="1.778" layer="96"/>
 </instance>
 <instance part="R9" gate="G$1" x="55.88" y="160.02" smashed="yes" rot="R180">
@@
 <attribute name="VALUE" x="45.72" y="172.72" size="1.778" layer="96" rot="R90"/>
 </instance>
-<instance part="J1" gate="G$1" x="15.24" y="154.94" smashed="yes" rot="MR0">
-<attribute name="VALUE" x="17.78" y="148.844" size="1.778" layer="96" rot="MR0"/>
-<attribute name="NAME" x="17.78" y="159.004" size="1.778" layer="96" rot="MR0"/>
-</instance>
 <instance part="GND8" gate="1" x="292.1" y="10.16" smashed="yes">
 <attribute name="VALUE" x="289.56" y="7.62" size="1.778" layer="96"/>
@@
 <instance part="GND27" gate="1" x="231.14" y="12.7" smashed="yes">
 <attribute name="VALUE" x="228.6" y="10.16" size="1.778" layer="96"/>
+</instance>
+<instance part="J2" gate="G$1" x="12.7" y="119.38" smashed="yes">
+<attribute name="NAME" x="7.62" y="124.46" size="1.778" layer="95"/>
+<attribute name="VALUE" x="7.62" y="114.3" size="1.778" layer="96" align="top-left"/>
+</instance>
+<instance part="J1" gate="G$1" x="12.7" y="157.48" smashed="yes">
+<attribute name="NAME" x="7.62" y="162.56" size="1.778" layer="95"/>
+<attribute name="VALUE" x="7.62" y="149.86" size="1.778" layer="96" align="top-left"/>
 </instance>
 </instances>
@@
 </segment>
 <segment>
-<wire x1="20.32" y1="152.4" x2="25.4" y2="152.4" width="0.1524" layer="91"/>
+<wire x1="22.86" y1="152.4" x2="25.4" y2="152.4" width="0.1524" layer="91"/>
 <pinref part="GND6" gate="1" pin="GND"/>
 <wire x1="25.4" y1="152.4" x2="25.4" y2="149.86" width="0.1524" layer="91"/>
-<pinref part="J1" gate="G$1" pin="1"/>
-</segment>
-<segment>
-<pinref part="J2" gate="G$1" pin="1"/>
+<pinref part="J1" gate="G$1" pin="SLEEVE"/>
+</segment>
+<segment>
 <pinref part="GND7" gate="1" pin="GND"/>
-<wire x1="20.32" y1="116.84" x2="22.86" y2="116.84" width="0.1524" layer="91"/>
-<wire x1="22.86" y1="116.84" x2="22.86" y2="114.3" width="0.1524" layer="91"/>
+<wire x1="22.86" y1="116.84" x2="25.4" y2="116.84" width="0.1524" layer="91"/>
+<wire x1="25.4" y1="116.84" x2="25.4" y2="114.3" width="0.1524" layer="91"/>
+<pinref part="J2" gate="G$1" pin="SLEEVE"/>
 </segment>
 <segment>
@@
 <pinref part="R7" gate="G$1" pin="1"/>
 <wire x1="45.72" y1="154.94" x2="40.64" y2="154.94" width="0.1524" layer="91"/>
-<pinref part="J1" gate="G$1" pin="3"/>
 <pinref part="R4" gate="G$1" pin="1"/>
-<wire x1="40.64" y1="154.94" x2="20.32" y2="154.94" width="0.1524" layer="91"/>
+<wire x1="40.64" y1="154.94" x2="25.4" y2="154.94" width="0.1524" layer="91"/>
 <wire x1="40.64" y1="162.56" x2="40.64" y2="154.94" width="0.1524" layer="91"/>
 <junction x="40.64" y="154.94"/>
+<pinref part="J1" gate="G$1" pin="TIP"/>
+<wire x1="22.86" y1="157.48" x2="25.4" y2="157.48" width="0.1524" layer="91"/>
+<wire x1="25.4" y1="157.48" x2="25.4" y2="154.94" width="0.1524" layer="91"/>
 </segment>
 </net>
@@
 <pinref part="C1" gate="G$1" pin="2"/>
 <wire x1="33.02" y1="121.92" x2="27.94" y2="121.92" width="0.1524" layer="91"/>
-<pinref part="J2" gate="G$1" pin="2"/>
 <pinref part="R3" gate="G$1" pin="1"/>
-<wire x1="27.94" y1="121.92" x2="20.32" y2="121.92" width="0.1524" layer="91"/>
+<wire x1="27.94" y1="121.92" x2="22.86" y2="121.92" width="0.1524" layer="91"/>
 <wire x1="27.94" y1="124.46" x2="27.94" y2="121.92" width="0.1524" layer="91"/>
 <junction x="27.94" y="121.92"/>
+<pinref part="J2" gate="G$1" pin="TIP"/>
 </segment>
 </net>
@@
 <net name="N$38" class="0">
 <segment>
-<pinref part="J1" gate="G$1" pin="2"/>
-<wire x1="20.32" y1="157.48" x2="22.86" y2="157.48" width="0.1524" layer="91"/>
-<wire x1="22.86" y1="157.48" x2="22.86" y2="160.02" width="0.1524" layer="91"/>
 <pinref part="S1" gate="-7" pin="2"/>
-<wire x1="22.86" y1="160.02" x2="25.4" y2="160.02" width="0.1524" layer="91"/>
+<pinref part="J1" gate="G$1" pin="RING"/>
+<wire x1="25.4" y1="160.02" x2="22.86" y2="160.02" width="0.1524" layer="91"/>
 </segment>
 </net>
@@
 </nets>
 </sheet>
-<sheet>
-<description>con</description>
-<plain>
-</plain>
-<instances>
-</instances>
-<busses>
-</busses>
-<nets>
-</nets>
-</sheet>
